File: CAN_Channel.kicad_sch (KiCad schematic)
At the start: 7 parts, among them J3 Conn_01x01, U2 TJA1051T-3

Commit message: updated pinout, begin layout
Parts:
- removed J3: Conn_01x01, Connector_PinHeader_2.54mm:PinHeader_1x01_P2.54mm_Vertical, symbol Connector_Generic:Conn_01x01
- renumbered C15 to C18, C13 to C19, C14 to C20, R6 to R21, U2 to U4
Connections:
- net GND: now also U4.8 (S)
Changed lines of the file:
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@@
 	(paper "A4")
+	(junction
+		(at 93.98 101.6)
+		(diameter 0)
+		(color 0 0 0 0)
+	)
 	(junction
 		(at 149.86 82.55)
@@
 	(wire
 		(pts
+			(xy 93.98 101.6) (xy 116.84 101.6)
+		)
+		(stroke
+			(width 0)
+			(type default)
+		)
+	)
+	(wire
+		(pts
 			(xy 101.6 85.09) (xy 104.14 85.09)
 		)
@@
 	(wire
 		(pts
+			(xy 93.98 95.25) (xy 93.98 101.6)
+		)
+		(stroke
+			(width 0)
+			(type default)
+		)
+	)
+	(wire
+		(pts
 			(xy 72.39 92.71) (xy 72.39 90.17)
 		)
@@
 	(wire
 		(pts
-			(xy 72.39 101.6) (xy 116.84 101.6)
+			(xy 72.39 101.6) (xy 93.98 101.6)
 		)
 		(stroke
@@
 		(dnp no)
 		(fields_autoplaced yes)
-		(property "Reference" "C13"
+		(property "Reference" "C19"
 			(at 140.97 77.4699 0)
 			(show_name no)
@@
 			(project "RSC-LV3-SwitchSense"
 				(path "/ea09e839-df61-4c3f-abdc-aa7ae2f772fe/bf939f33-0653-4b59-bd63-3496752c5dd5/4645bb46-e9fc-4e0d-92f5-2f289dd6d3ff"
-					(reference "C13")
+					(reference "C19")
 					(unit 1)
 				)
@@
 		(dnp no)
 		(fields_autoplaced yes)
-		(property "Reference" "U2"
+		(property "Reference" "U4"
 			(at 118.9833 77.47 0)
 			(show_name no)
@@
 			(project "RSC-LV3-SwitchSense"
 				(path "/ea09e839-df61-4c3f-abdc-aa7ae2f772fe/bf939f33-0653-4b59-bd63-3496752c5dd5/4645bb46-e9fc-4e0d-92f5-2f289dd6d3ff"
-					(reference "U2")
+					(reference "U4")
 					(unit 1)
 				)
@@
 		(dnp no)
 		(fields_autoplaced yes)
-		(property "Reference" "R6"
+		(property "Reference" "R21"
 			(at 179.07 85.09 90)
 			(show_name no)
@@
 			(project "RSC-LV3-SwitchSense"
 				(path "/ea09e839-df61-4c3f-abdc-aa7ae2f772fe/bf939f33-0653-4b59-bd63-3496752c5dd5/4645bb46-e9fc-4e0d-92f5-2f289dd6d3ff"
-					(reference "R6")
+					(reference "R21")
 					(unit 1)
 				)
@@
 		(dnp no)
 		(fields_autoplaced yes)
-		(property "Reference" "#PWR018"
+		(property "Reference" "#PWR043"
 			(at 149.86 77.47 0)
 			(hide yes)
@@
 			(project "RSC-LV3-SwitchSense"
 				(path "/ea09e839-df61-4c3f-abdc-aa7ae2f772fe/bf939f33-0653-4b59-bd63-3496752c5dd5/4645bb46-e9fc-4e0d-92f5-2f289dd6d3ff"
-					(reference "#PWR018")
+					(reference "#PWR043")
 					(unit 1)
 				)
@@
 		(dnp no)
 		(fields_autoplaced yes)
-		(property "Reference" "C14"
+		(property "Reference" "C20"
 			(at 153.67 77.4699 0)
 			(show_name no)
@@
 			(project "RSC-LV3-SwitchSense"
 				(path "/ea09e839-df61-4c3f-abdc-aa7ae2f772fe/bf939f33-0653-4b59-bd63-3496752c5dd5/4645bb46-e9fc-4e0d-92f5-2f289dd6d3ff"
-					(reference "C14")
+					(reference "C20")
 					(unit 1)
 				)
@@
 		(dnp no)
 		(fields_autoplaced yes)
-		(property "Reference" "#PWR019"
+		(property "Reference" "#PWR041"
 			(at 72.39 93.98 0)
 			(hide yes)
@@
 			(project "RSC-LV3-SwitchSense"
 				(path "/ea09e839-df61-4c3f-abdc-aa7ae2f772fe/bf939f33-0653-4b59-bd63-3496752c5dd5/4645bb46-e9fc-4e0d-92f5-2f289dd6d3ff"
-					(reference "#PWR019")
+					(reference "#PWR041")
 					(unit 1)
 				)
@@
 		(dnp no)
 		(fields_autoplaced yes)
-		(property "Reference" "C15"
+		(property "Reference" "C18"
 			(at 76.2 95.2499 0)
 			(show_name no)
@@
 			(project "RSC-LV3-SwitchSense"
 				(path "/ea09e839-df61-4c3f-abdc-aa7ae2f772fe/bf939f33-0653-4b59-bd63-3496752c5dd5/4645bb46-e9fc-4e0d-92f5-2f289dd6d3ff"
-					(reference "C15")
+					(reference "C18")
 					(unit 1)
 				)
@@
 	)
 	(symbol
-		(lib_id "Connector_Generic:Conn_01x01")
-		(at 88.9 95.25 180)
-		(unit 1)
-		(body_style 1)
-		(exclude_from_sim no)
-		(in_bom yes)
-		(on_board yes)
-		(in_pos_files yes)
-		(dnp no)
-		(fields_autoplaced yes)
-		(property "Reference" "J3"
-			(at 88.9 88.9 0)
-			(show_name no)
-			(do_not_autoplace no)
-			(effects
-				(font
-					(size 1.27 1.27)
-				)
-			)
-		)
-		(property "Value" "Conn_01x01"
-			(at 88.9 91.44 0)
-			(show_name no)
-			(do_not_autoplace no)
-			(effects
-				(font
-					(size 1.27 1.27)
-				)
-			)
-		)
-		(property "Footprint" "Connector_PinHeader_2.54mm:PinHeader_1x01_P2.54mm_Vertical"
-			(at 88.9 95.25 0)
-			(hide yes)
-			(show_name no)
-			(do_not_autoplace no)
-			(effects
-				(font
-					(size 1.27 1.27)
-				)
-			)
-		)
-		(property "Datasheet" ""
-			(at 88.9 95.25 0)
-			(hide yes)
-			(show_name no)
-			(do_not_autoplace no)
-			(effects
-				(font
-					(size 1.27 1.27)
-				)
-			)
-		)
-		(property "Description" "Generic connector, single row, 01x01, script generated (kicad-library-utils/schlib/autogen/connector/)"
-			(at 88.9 95.25 0)
-			(hide yes)
-			(show_name no)
-			(do_not_autoplace no)
-			(effects
-				(font
-					(size 1.27 1.27)
-				)
-			)
-		)
-		(pin "1"
-		)
-		(instances
-			(project "RSC-LV3-SwitchSense"
-				(path "/ea09e839-df61-4c3f-abdc-aa7ae2f772fe/bf939f33-0653-4b59-bd63-3496752c5dd5/4645bb46-e9fc-4e0d-92f5-2f289dd6d3ff"
-					(reference "J3")
-					(unit 1)
-				)
-			)
-		)
-	)
-	(symbol
 		(lib_id "power:GND")
 		(at 116.84 101.6 0)
@@
 		(dnp no)
 		(fields_autoplaced yes)
-		(property "Reference" "#PWR020"
+		(property "Reference" "#PWR042"
 			(at 116.84 107.95 0)
 			(hide yes)
@@
 			(project "RSC-LV3-SwitchSense"
 				(path "/ea09e839-df61-4c3f-abdc-aa7ae2f772fe/bf939f33-0653-4b59-bd63-3496752c5dd5/4645bb46-e9fc-4e0d-92f5-2f289dd6d3ff"
-					(reference "#PWR020")
+					(reference "#PWR042")
 					(unit 1)
 				)

Commit message: r0 final
Parts:
- renumbered C18 to C24, C19 to C25, C20 to C26, R21 to R31
Changed lines of the file:
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@@
 		(dnp no)
 		(fields_autoplaced yes)
-		(property "Reference" "C19"
+		(property "Reference" "C25"
 			(at 140.97 77.4699 0)
 			(show_name no)
@@
 			(project "RSC-LV3-HVBPS"
 				(path "/ea09e839-df61-4c3f-abdc-aa7ae2f772fe/bf939f33-0653-4b59-bd63-3496752c5dd5/4645bb46-e9fc-4e0d-92f5-2f289dd6d3ff"
-					(reference "C19")
+					(reference "C25")
 					(unit 1)
 				)
 				(path "/ea09e839-df61-4c3f-abdc-aa7ae2f772fe/bf939f33-0653-4b59-bd63-3496752c5dd5/ef23ee7b-7f39-46c1-8aad-e04e597a3661"
-					(reference "C33")
+					(reference "C28")
 					(unit 1)
 				)
@@
 		(dnp no)
 		(fields_autoplaced yes)
-		(property "Reference" "R21"
+		(property "Reference" "R31"
 			(at 179.07 85.09 90)
 			(show_name no)
@@
 			(project "RSC-LV3-HVBPS"
 				(path "/ea09e839-df61-4c3f-abdc-aa7ae2f772fe/bf939f33-0653-4b59-bd63-3496752c5dd5/4645bb46-e9fc-4e0d-92f5-2f289dd6d3ff"
-					(reference "R21")
+					(reference "R31")
 					(unit 1)
 				)
 				(path "/ea09e839-df61-4c3f-abdc-aa7ae2f772fe/bf939f33-0653-4b59-bd63-3496752c5dd5/ef23ee7b-7f39-46c1-8aad-e04e597a3661"
-					(reference "R62")
+					(reference "R32")
 					(unit 1)
 				)
@@
 		(dnp no)
 		(fields_autoplaced yes)
-		(property "Reference" "#PWR043"
+		(property "Reference" "#PWR062"
 			(at 149.86 77.47 0)
 			(hide yes)
@@
 			(project "RSC-LV3-HVBPS"
 				(path "/ea09e839-df61-4c3f-abdc-aa7ae2f772fe/bf939f33-0653-4b59-bd63-3496752c5dd5/4645bb46-e9fc-4e0d-92f5-2f289dd6d3ff"
-					(reference "#PWR043")
+					(reference "#PWR062")
 					(unit 1)
 				)
 				(path "/ea09e839-df61-4c3f-abdc-aa7ae2f772fe/bf939f33-0653-4b59-bd63-3496752c5dd5/ef23ee7b-7f39-46c1-8aad-e04e597a3661"
-					(reference "#PWR077")
+					(reference "#PWR065")
 					(unit 1)
 				)
@@
 		(dnp no)
 		(fields_autoplaced yes)
-		(property "Reference" "C20"
+		(property "Reference" "C26"
 			(at 153.67 77.4699 0)
 			(show_name no)
@@
 			(project "RSC-LV3-HVBPS"
 				(path "/ea09e839-df61-4c3f-abdc-aa7ae2f772fe/bf939f33-0653-4b59-bd63-3496752c5dd5/4645bb46-e9fc-4e0d-92f5-2f289dd6d3ff"
-					(reference "C20")
+					(reference "C26")
 					(unit 1)
 				)
 				(path "/ea09e839-df61-4c3f-abdc-aa7ae2f772fe/bf939f33-0653-4b59-bd63-3496752c5dd5/ef23ee7b-7f39-46c1-8aad-e04e597a3661"
-					(reference "C34")
+					(reference "C29")
 					(unit 1)
 				)
@@
 		(dnp no)
 		(fields_autoplaced yes)
-		(property "Reference" "#PWR041"
+		(property "Reference" "#PWR060"
 			(at 72.39 93.98 0)
 			(hide yes)
@@
 			(project "RSC-LV3-HVBPS"
 				(path "/ea09e839-df61-4c3f-abdc-aa7ae2f772fe/bf939f33-0653-4b59-bd63-3496752c5dd5/4645bb46-e9fc-4e0d-92f5-2f289dd6d3ff"
-					(reference "#PWR041")
+					(reference "#PWR060")
 					(unit 1)
 				)
 				(path "/ea09e839-df61-4c3f-abdc-aa7ae2f772fe/bf939f33-0653-4b59-bd63-3496752c5dd5/ef23ee7b-7f39-46c1-8aad-e04e597a3661"
-					(reference "#PWR075")
+					(reference "#PWR063")
 					(unit 1)
 				)
@@
 		(dnp no)
 		(fields_autoplaced yes)
-		(property "Reference" "C18"
+		(property "Reference" "C24"
 			(at 76.2 95.2499 0)
 			(show_name no)
@@
 			(project "RSC-LV3-HVBPS"
 				(path "/ea09e839-df61-4c3f-abdc-aa7ae2f772fe/bf939f33-0653-4b59-bd63-3496752c5dd5/4645bb46-e9fc-4e0d-92f5-2f289dd6d3ff"
-					(reference "C18")
+					(reference "C24")
 					(unit 1)
 				)
 				(path "/ea09e839-df61-4c3f-abdc-aa7ae2f772fe/bf939f33-0653-4b59-bd63-3496752c5dd5/ef23ee7b-7f39-46c1-8aad-e04e597a3661"
-					(reference "C32")
+					(reference "C27")
 					(unit 1)
 				)
@@
 		(dnp no)
 		(fields_autoplaced yes)
-		(property "Reference" "#PWR042"
+		(property "Reference" "#PWR061"
 			(at 116.84 107.95 0)
 			(hide yes)
@@
 			(project "RSC-LV3-HVBPS"
 				(path "/ea09e839-df61-4c3f-abdc-aa7ae2f772fe/bf939f33-0653-4b59-bd63-3496752c5dd5/4645bb46-e9fc-4e0d-92f5-2f289dd6d3ff"
-					(reference "#PWR042")
+					(reference "#PWR061")
 					(unit 1)
 				)
 				(path "/ea09e839-df61-4c3f-abdc-aa7ae2f772fe/bf939f33-0653-4b59-bd63-3496752c5dd5/ef23ee7b-7f39-46c1-8aad-e04e597a3661"
-					(reference "#PWR076")
-					(unit 1)
-				)
+					(reference "#PWR064")
+					(unit 1)
+				)
