File: Indicator_LED.kicad_sch (KiCad schematic)
At the start: 0 parts

Commit message: updated pinout, begin layout
Parts:
- added D2: LED_RGB, LED_SMD:LED_RGB_5050-6, symbol Device:LED_RGB
- added R6, R7: 50, Resistor_SMD:R_0603_1608Metric_Pad0.98x0.95mm_HandSolder, symbol Device:R
- added R8: 120, Resistor_SMD:R_0603_1608Metric_Pad0.98x0.95mm_HandSolder, symbol Device:R
Connections:
- new net: D2.2 (GK), R7.2
- new net: D2.3 (BK), R6.2
- new net: D2.1 (RK), R8.2
- new net B+: D2.4 (BA)
- new net G+: D2.5 (GA)
- new net GND: R6.1, R7.1, R8.1
- new net R+: D2.6 (RA)

Commit message: r0 final
Parts:
- renumbered D2 to D6, R6 to R16, R7 to R17, R8 to R18
Changed lines of the file:
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@@
 		(in_pos_files yes)
 		(dnp no)
-		(property "Reference" "R7"
+		(property "Reference" "R17"
 			(at 135.89 87.6299 0)
 			(show_name no)
@@
 			(project "RSC-LV3-HVBPS"
 				(path "/ea09e839-df61-4c3f-abdc-aa7ae2f772fe/4aa7ee16-37d7-4a92-b053-2235cd7f2d7b/0ba67f90-927b-4a9b-b1dc-32a9d85f8a8c"
-					(reference "R7")
+					(reference "R17")
 					(unit 1)
 				)
 				(path "/ea09e839-df61-4c3f-abdc-aa7ae2f772fe/4aa7ee16-37d7-4a92-b053-2235cd7f2d7b/61bc5597-943d-40ea-9229-119231165e79"
-					(reference "R10")
+					(reference "R20")
 					(unit 1)
 				)
@@
 		(in_pos_files yes)
 		(dnp no)
-		(property "Reference" "R6"
+		(property "Reference" "R16"
 			(at 128.27 92.7099 0)
 			(show_name no)
@@
 			(project "RSC-LV3-HVBPS"
 				(path "/ea09e839-df61-4c3f-abdc-aa7ae2f772fe/4aa7ee16-37d7-4a92-b053-2235cd7f2d7b/0ba67f90-927b-4a9b-b1dc-32a9d85f8a8c"
-					(reference "R6")
+					(reference "R16")
 					(unit 1)
 				)
 				(path "/ea09e839-df61-4c3f-abdc-aa7ae2f772fe/4aa7ee16-37d7-4a92-b053-2235cd7f2d7b/61bc5597-943d-40ea-9229-119231165e79"
-					(reference "R9")
+					(reference "R19")
 					(unit 1)
 				)
@@
 		(in_pos_files yes)
 		(dnp no)
-		(property "Reference" "R8"
+		(property "Reference" "R18"
 			(at 143.51 82.5499 0)
 			(show_name no)
@@
 			(project "RSC-LV3-HVBPS"
 				(path "/ea09e839-df61-4c3f-abdc-aa7ae2f772fe/4aa7ee16-37d7-4a92-b053-2235cd7f2d7b/0ba67f90-927b-4a9b-b1dc-32a9d85f8a8c"
-					(reference "R8")
+					(reference "R18")
 					(unit 1)
 				)
 				(path "/ea09e839-df61-4c3f-abdc-aa7ae2f772fe/4aa7ee16-37d7-4a92-b053-2235cd7f2d7b/61bc5597-943d-40ea-9229-119231165e79"
-					(reference "R11")
+					(reference "R21")
 					(unit 1)
 				)
@@
 		(dnp no)
 		(fields_autoplaced yes)
-		(property "Reference" "D2"
+		(property "Reference" "D6"
 			(at 118.11 71.12 0)
 			(show_name no)
@@
 			(project "RSC-LV3-HVBPS"
 				(path "/ea09e839-df61-4c3f-abdc-aa7ae2f772fe/4aa7ee16-37d7-4a92-b053-2235cd7f2d7b/0ba67f90-927b-4a9b-b1dc-32a9d85f8a8c"
-					(reference "D2")
+					(reference "D6")
 					(unit 1)
 				)
 				(path "/ea09e839-df61-4c3f-abdc-aa7ae2f772fe/4aa7ee16-37d7-4a92-b053-2235cd7f2d7b/61bc5597-943d-40ea-9229-119231165e79"
-					(reference "D3")
+					(reference "D7")
 					(unit 1)
 				)
@@
 		(dnp no)
 		(fields_autoplaced yes)
-		(property "Reference" "#PWR019"
+		(property "Reference" "#PWR037"
 			(at 125.73 104.14 0)
 			(hide yes)
@@
 			(project "RSC-LV3-HVBPS"
 				(path "/ea09e839-df61-4c3f-abdc-aa7ae2f772fe/4aa7ee16-37d7-4a92-b053-2235cd7f2d7b/0ba67f90-927b-4a9b-b1dc-32a9d85f8a8c"
-					(reference "#PWR019")
+					(reference "#PWR037")
 					(unit 1)
 				)
 				(path "/ea09e839-df61-4c3f-abdc-aa7ae2f772fe/4aa7ee16-37d7-4a92-b053-2235cd7f2d7b/61bc5597-943d-40ea-9229-119231165e79"
-					(reference "#PWR020")
-					(unit 1)
-				)
+					(reference "#PWR038")
+					(unit 1)
+				)
